File: PCB/Main/Cinder.kicad_pcb (KiCad board)
At the start: 2 copper layers, 60 x 80 mm, 22 parts, among them J1 -, J2 +, J3 +, J4 -, Q1 IPD33CN10N G, Q2 IPD33CN10N G, SW1 SW_Push, SW2 SW_Push, SW3 SW_Push, SW9 EC11E09244BS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

Commit message: Update
Parts:
- added C1: 0.01uF, Capacitor_SMD:C_1206_3216Metric_Pad1.33x1.80mm_HandSolder, F.Cu at (147.2, 67.5)
- added C2: 0.1uF, Capacitor_SMD:C_1206_3216Metric_Pad1.33x1.80mm_HandSolder, F.Cu at (142.2, 70.8)
- added C3: 0.1uF, Capacitor_SMD:C_1206_3216Metric_Pad1.33x1.80mm_HandSolder, F.Cu at (150.5, 54.8)
- added C4: 0.1uF, Capacitor_SMD:C_1206_3216Metric_Pad1.33x1.80mm_HandSolder, F.Cu at (150.5, 52.0)
- added C5: 0.47uF, Capacitor_SMD:C_1206_3216Metric_Pad1.33x1.80mm_HandSolder, F.Cu at (133.8, 53.2)
- added J5: Stepper, Connector_PinHeader_2.54mm:PinHeader_1x04_P2.54mm_Vertical, B.Cu at (128.0, 79.5)
- added J6: SHT40, Connector_PinHeader_2.54mm:PinHeader_1x04_P2.54mm_Vertical, F.Cu at (128.0, 65.2)
- added J7: IR sensor, Connector_PinHeader_2.54mm:PinHeader_1x04_P2.54mm_Vertical, F.Cu at (128.0, 61.0)
- added R10: 0.2, Resistor_SMD:R_1206_3216Metric_Pad1.30x1.75mm_HandSolder, F.Cu at (151.0, 67.0)
- added R11: 0.2, Resistor_SMD:R_1206_3216Metric_Pad1.30x1.75mm_HandSolder, F.Cu at (154.5, 67.0)
- added R12: 2.2K, Resistor_SMD:R_1206_3216Metric_Pad1.30x1.75mm_HandSolder, F.Cu at (139.0, 53.2)
- added R13: 4.7K, Resistor_SMD:R_1206_3216Metric_Pad1.30x1.75mm_HandSolder, F.Cu at (144.2, 55.2)
- added R15: 10K, Resistor_SMD:R_1206_3216Metric_Pad1.30x1.75mm_HandSolder, F.Cu at (137.0, 55.8)
- added R16: 10K, Resistor_SMD:R_1206_3216Metric_Pad1.30x1.75mm_HandSolder, F.Cu at (139.5, 88.0)
- added R17: 10K, Resistor_SMD:R_1206_3216Metric_Pad1.30x1.75mm_HandSolder, F.Cu at (145.2, 88.0)
- added R9: 1M, Resistor_SMD:R_1206_3216Metric_Pad1.30x1.75mm_HandSolder, F.Cu at (142.2, 68.2)
- added U5: DRV8825PWPR, LCSC:HTSSOP-28_L9.7-W4.4-P0.65-LS6.4-BL-EP5.5, F.Cu at (142.1, 61.8)
- added U6: 100uF 25V, LCSC:CAP-SMD_BD6.3-L6.6-W6.6-LS7.2-FD-1, B.Cu at (142.0, 61.3)
- J1: value - -> Heater -
- J2: value + -> Heater +
- J3: value + -> Fan +
- J4: value - -> Fan -
- Q1, Q2, R1, R2, R3, R4: moved to F.Cu
- moved R2 30.4 mm to (157.5, 67.8)
- moved R1 28.8 mm to (156.5, 61.5), turned to 0 degrees
- moved R4 22.5 mm to (156.2, 58.8)
- moved R8 14.9 mm to (152.8, 86.0), turned to 0 degrees
- moved U1 9.81 mm to (142.2, 62.5)
- moved J2 9.73 mm to (182.0, 67.3)
- moved J3 9.73 mm to (182.0, 72.3)
- moved J4 9.73 mm to (182.0, 77.3)
- moved J1 9.73 mm to (182.0, 62.7)
- moved Q2 9.28 mm to (164.2, 76.8)
- moved R3 8.92 mm to (154.5, 75.0)
- moved U3 8.88 mm to (165.0, 53.0)
- moved R7 7.70 mm to (156.8, 94.8), turned to 0 degrees
- moved Q1 7.67 mm to (164.2, 69.0)
- moved R5 5.30 mm to (156.8, 97.2), turned to 0 degrees
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Connections:
- net Net-(U1-GP0) renamed IR_SDA
- net Net-(U1-GP1) renamed IR_SCL
- R1 pad 1: Net-(U1-GP2) -> HAETER
- R2 pad 1: Net-(U1-GP3) -> FAN
- R5 pad 1: SW1 -> SW2
- R6 pad 1: SW2 -> SW1
- SW1 pad 2: SW2 -> SW1
- SW2 pad 2: SW1 -> SW2
- U1 pad 13: unconnected-(U1-GP12-Pad13) -> SW1
- U1 pad 14: unconnected-(U1-GP13-Pad14) -> SW2
- U1 pad 15: SW4 -> SW3
- U1 pad 16: SW3 -> SW4
- U1 pad 17: SW2 -> EC2
- U1 pad 18: SW1 -> EC1
- U1 pad 19: EC2 -> FAN
- U1 pad 20: EC1 -> HAETER
- U1 pad 3: Net-(U1-GP2) -> nFault
- U1 pad 4: Net-(U1-GP3) -> DIR
- U1 pad 5: unconnected-(U1-GP4-Pad5) -> ENABLE
- U1 pad 6: unconnected-(U1-GP5-Pad6) -> STEP
- U1 pad 7: unconnected-(U1-GP6-Pad7) -> MODE0
- U1 pad 8: unconnected-(U1-GP7-Pad8) -> MODE1
- U1 pad 9: unconnected-(U1-GP8-Pad9) -> MODE2
Routing:
- net +19V: track 56.5 -> 128.3 mm, vias 0 -> 4
- net Net-(J5-Pin_4): track 0.00 -> 52.3 mm
- net Net-(J5-Pin_3): track 0.00 -> 45.3 mm
- net Net-(Q1-G): track 53.1 -> 9.39 mm
- net Net-(J5-Pin_2): track 0.00 -> 42.5 mm
- net Net-(J5-Pin_1): track 0.00 -> 37.3 mm
- net Net-(Q2-G): track 44.8 -> 10.2 mm
- net +5V: track 70.2 -> 100.1 mm, vias 1 -> 3
- net SW2: track 99.8 -> 82.0 mm
- net Net-(U5-VCP): track 0.00 -> 17.2 mm
- net IR_SCL: track 45.5 -> 62.6 mm
- net Net-(J1-Pin_1): track 0.00 -> 17.1 mm
- net SW4: track 31.0 -> 46.1 mm, vias 2 -> 0
- net GND: track 2.25 -> 16.0 mm, vias 45 -> 14
- net Net-(U1-GP3): track 12.2 -> 0.00 mm, vias 2 -> 0
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- removed copper zone on F.Cu, net +19V
- removed copper zone on B.Cu, net Net-(J1-Pin_1)
Other:
- board size 60 x 80 mm -> 60 x 90 mm
- board text added: "IR sensor"
- board text added: "SHT40"
- board text added: "Stepper"
